File: hummingbird_routing.kicad_pcb (KiCad board)
At the start: 2 copper layers, 109.3 x 81.4 mm, 16 parts

Commit message: Added On/Off Switches
Parts:
- removed MCU1: , nicenano
- removed S1, S10, S11, S12, S13, S14, S15, S2, S3, S4, S5, S6, S7, S8, S9: , PG1350
Routing:
- net matrix_pinky_home: track 126.3 -> 0.00 mm
- net matrix_pinky_top: track 124.3 -> 0.00 mm
- net matrix_ring_bottom: track 104.9 -> 0.00 mm
- net matrix_ring_top: track 87.5 -> 0.00 mm
- net matrix_middle_bottom: track 84.1 -> 0.00 mm
- net matrix_ring_home: track 81.8 -> 0.00 mm
- net matrix_middle_top: track 68.9 -> 0.00 mm
- net matrix_index_bottom: track 63.9 -> 0.00 mm
- net matrix_middle_home: track 62.8 -> 0.00 mm
- net matrix_index_top: track 52.9 -> 0.00 mm
- net matrix_index_home: track 46.5 -> 0.00 mm
- net thumb_tucky: track 38.8 -> 0.00 mm
- net matrix_inner_top: track 35.1 -> 0.00 mm
- net matrix_inner_home: track 28.8 -> 0.00 mm
- net thumb_reachy: track 24.6 -> 0.00 mm
Other:
- copper layers 2 -> 0
Changed lines of the file:
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@@
 	(generator "pcbnew")
 	(generator_version "8.0")
-	(general
 		(thickness 1.6)
 		(legacy_teardrops no)
@@
 		(rev "v1.0.0")
 		(company "Unknown")
-	)
 	(layers
 		(0 "F.Cu" signal)
